File: mainboard_ESP32 DevBoard.sch (EAGLE design)
At the start: 44 parts, among them K1 AQH213, T1 2N2222, U1 LM833N, U2 ILD620GB, U3 DG419DJ-L, U4 ESP32-DOIT-V1, U5 TEMP-HUM-SENSOR-DHT22, X1 JST-XH-02-PIN-LONG-PAD, X2 JST-XH-04-PIN-LONG-PAD, X3 1751293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

Commit message: Added pullup resistors for I2C bus
Parts:
- added R14, R20: 2.4K, Passive:RESISTORL
Connections:
- net +3V3: now also R14.2, R20.2
- net SCL: now also R14.1
- net SDA: now also R20.1
Changed lines of the file:
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@@
 <part name="GND1" library="supply1" library_urn="urn:adsk.eagle:library:371" deviceset="GND" device=""/>
 <part name="MOV1" library="EVSE" deviceset="MOV-07D471K" device=""/>
+<part name="R14" library="Passive" deviceset="RESISTOR" device="L" value="2.4K"/>
+<part name="R20" library="Passive" deviceset="RESISTOR" device="L" value="2.4K"/>
+<part name="+3V3" library="supply1" library_urn="urn:adsk.eagle:library:371" deviceset="+3V3" device=""/>
+<part name="+3V7" library="supply1" library_urn="urn:adsk.eagle:library:371" deviceset="+3V3" device=""/>
 </parts>
 <sheets>
@@
 <attribute name="VALUE" x="144.78" y="-46.99" size="1.778" layer="96" align="top-left"/>
 </instance>
+<instance part="R14" gate="G$1" x="210.82" y="139.7" smashed="yes" rot="R90">
+<attribute name="NAME" x="209.3214" y="135.89" size="1.778" layer="95" rot="R90"/>
+<attribute name="VALUE" x="214.122" y="135.89" size="1.778" layer="96" rot="R90"/>
+</instance>
+<instance part="R20" gate="G$1" x="220.98" y="139.7" smashed="yes" rot="R90">
+<attribute name="NAME" x="219.4814" y="135.89" size="1.778" layer="95" rot="R90"/>
+<attribute name="VALUE" x="224.282" y="135.89" size="1.778" layer="96" rot="R90"/>
+</instance>
+<instance part="+3V3" gate="G$1" x="210.82" y="149.86" smashed="yes">
+<attribute name="VALUE" x="205.74" y="149.86" size="1.778" layer="96" rot="R270"/>
+</instance>
+<instance part="+3V7" gate="G$1" x="220.98" y="149.86" smashed="yes">
+<attribute name="VALUE" x="215.9" y="149.86" size="1.778" layer="96" rot="R270"/>
+</instance>
 </instances>
 <busses>
@@
 <junction x="99.06" y="43.18"/>
 </segment>
+<segment>
+<pinref part="R14" gate="G$1" pin="2"/>
+<wire x1="210.82" y1="144.78" x2="210.82" y2="147.32" width="0.1524" layer="91"/>
+<pinref part="+3V3" gate="G$1" pin="+3V3"/>
+</segment>
+<segment>
+<pinref part="R20" gate="G$1" pin="2"/>
+<wire x1="220.98" y1="144.78" x2="220.98" y2="147.32" width="0.1524" layer="91"/>
+<pinref part="+3V7" gate="G$1" pin="+3V3"/>
+</segment>
 </net>
 <net name="+12V" class="0">
@@
 <label x="7.62" y="66.04" size="1.27" layer="95" rot="R180" xref="yes"/>
 </segment>
+<segment>
+<pinref part="R20" gate="G$1" pin="1"/>
+<wire x1="220.98" y1="134.62" x2="220.98" y2="132.08" width="0.1524" layer="91"/>
+<label x="220.98" y="132.08" size="1.778" layer="95" rot="R270" xref="yes"/>
+</segment>
 </net>
 <net name="SCL" class="0">
@@
 <label x="7.62" y="63.5" size="1.27" layer="95" rot="R180" xref="yes"/>
 </segment>
-</net>
+<segment>
+<pinref part="R14" gate="G$1" pin="1"/>
+<wire x1="210.82" y1="134.62" x2="210.82" y2="132.08" width="0.1524" layer="91"/>
+<label x="210.82" y="132.08" size="1.778" layer="95" rot="R270" xref="yes"/>
+</segment>
+</net>
